File: Hardware/MicroMouse.sch (KiCad schematic (older format))
At the start: 1 part

Commit message: Added Power Managemen Dsign
Parts:
- added C? (x3): 10uF, symbol Device:C_Small
- added C?: 1700pF, symbol Device:C_Small
- added C?: DNP, symbol Device:C_Small
- added C? (x2): 1uF, symbol Device:C_Small
- added C?: 33nF, symbol Device:C_Small
- added D?: MBRA210LT, symbol Device:D_Schottky_Small_ALT
- added L? (x2): 744878004, symbol Mice_Sym:744878004
- added R?: 8.2k, symbol Device:R_Small
- added R?: 0R, symbol Device:R_Small
- added R? (x2): 10k, symbol Device:R_Small
- added R?: DNP, symbol Device:R_Small
- added R?: 12k, symbol Device:R_Small
- added R?: 30.5k, symbol Device:R_Small
Connections:
- net at U?.1 (COMP): now also C?.1, R?.1
- net at U?.2 (FB): now also R?.1, R?.2
- net at U?.3 (EN): now also R?.1, R?.2
- net GND: now reaches U?.4 (GND)
- net GND: now also C?.2, C?.2, C?.2, C?.2, C?.2, C?.2, C?.2, L?.4, R?.2, R?.2, R?.2
- net at U?.5 (SW): now also C?.2, L?.2
- net +BATT: now reaches U?.6 (VIN)
- net +BATT: now also C?.1, L?.1, R?.1, R?.1
- net at U?.7 (FREQ): now also R?.1, R?.2
- net at U?.8 (SS): now also C?.1
- new net: C?.1, D?.2 (A), L?.3
- new net: C?.1, R?.2
- new net +5V: C?.1, C?.1, C?.1, D?.1 (K), R?.1
Other:
- note added: "Power Management"
- moved on the sheet: U?

Commit message: Update hardware design
Parts:
- added C? (x2): 22pF, symbol Device:C_Small
- added C?: 1uF, symbol Device:C_Small
- added C?: 0.1uF, symbol Device:C_Small
- added D?: MMSZ5231B-7-F, symbol Device:D_Zener_Small_ALT
- added FB?: 120R, symbol Device:Ferrite_Bead_Small
- added J?: 68024-102HLF, symbol Connector:Conn_01x02_Male
- added J?: TSW-106-25-S-S-RA, symbol Connector:Conn_01x06_Male
- added J?: 78511-106HLF, symbol Connector:Conn_01x06_Male
- added Q?: NXV75UPR, symbol Device:Q_PMOS_GSD
- added R? (x2): 1k, symbol Device:R_Small
- added R?: 10k, symbol Device:R_Small
- added R?: 220k, symbol Device:R_Small
- added SW?: L101011MS02Q, symbol Switch:SW_DIP_x01
- added SW? (x7): SPST, symbol Mice_Sym:SPST
- added U? (x3): PIC16F886-E_SO, symbol Mice_Sym:PIC16F886-E_SO
- added Y?: 32.768KHZ, symbol Device:Crystal_Small
Connections:
- net +5V: now also C?.1, C?.1, FB?.1, J?.2 (Pin_2), J?.2 (Pin_2), R?.2, U?.20 (VDD); no longer C?.1, C?.1, C?.1, D?.1 (K), R?.1
- net +BATT: now also J?.1 (Pin_1), SW?.1; no longer C?.1, L?.1, R?.1, R?.1, U?.6 (VIN)
- net GND: now also C?.1, C?.1, C?.2, C?.2, J?.2 (Pin_2), J?.3 (Pin_3), J?.3 (Pin_3), R?.2, SW?.1 (A), SW?.2 (A), U?.19 (VSS), U?.8 (VSS)
- new net: Q?.3 (D), SW?.2
- new net: D?.2 (A), Q?.1 (G), R?.1
- new net: R?.2, U?.11 (RC0/T1OSO/T1CK1)
- new net: C?.2, U?.12 (RC1/T1OSI/CCP2), Y?.2
- new net: R?.1, R?.2, SW?.3 (B), SW?.4 (B)
- new net: C?.2, R?.1, Y?.1
- new net: J?.5 (Pin_5), U?.14 (RC3/SCK/SCL)
- new net: J?.4 (Pin_4), U?.15 (RC4/SDI/SDA)
- new net: J?.6 (Pin_6), U?.17 (RC6/TX/CK)
- new net: J?.1 (Pin_1), U?.18 (RC7/RX/DT)
- new net +5P: C?.1, C?.1, C?.1, D?.1 (K), FB?.2, R?.1
- new net Aux: J?.6 (Pin_6)
- new net C1: SW?.3 (B), SW?.3 (B), SW?.4 (B), SW?.4 (B), U?.22 (P1C/AN10/RB1)
- new net C2: SW?.3 (B), SW?.3 (B), SW?.4 (B), SW?.4 (B), U?.13 (RC2/P1A/CCP1)
- new net C3: SW?.3 (B), SW?.3 (B), SW?.4 (B), SW?.4 (B), U?.16 (RC5/SDO)
- new net R1: J?.4 (Pin_4), SW?.1 (A), SW?.1 (A), SW?.1 (A), SW?.2 (A), SW?.2 (A), SW?.2 (A), U?.28 (ICSPDAT/RB7)
- new net R2: J?.5 (Pin_5), SW?.1 (A), SW?.1 (A), SW?.1 (A), SW?.2 (A), SW?.2 (A), SW?.2 (A), U?.27 (ICSPCLK/RB6)
- new net VCC: C?.1, D?.1 (K), L?.1, Q?.2 (S), R?.1, R?.1, U?.6 (VIN)
- new net Vpp: J?.1 (Pin_1), R?.1, U?.1 (RE3/~MCLR~/Vpp)
Other:
- note added: "MCU Interfaces"
- note added: "MCU Power"
- moved on the sheet: C?, D?, L?A, L?B, R?, U?
